File: 89c52board.kicad_pcb (KiCad board)
At the start: 2 copper layers, 99.1 x 99.1 mm, 47 parts, among them J1 Anodes, J11 P0.6-7, J12 P1.4-7, J13 P3.6-7, J2 Anodes, J3 Cathodes, J4 RTC board, J5 ISP, J6 12VDC, Q1 NPN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

Commit message: Cosmetic: swap C2 and C4 labels to better reflect their positions on board
Parts:
- renumbered C4 to C2, C2 to C4

Commit message: More suitable values for I2C pullup resistors and digit driver transistor base resistor. Board unchanged
Parts:
- R1: value 1k -> 4k7
- R7, R8: value 10k -> 4k7
